File: ROS2_final_project_PCB.kicad_pcb (KiCad board)
At the start: 2 copper layers, 18 parts, among them J1 Conn_01x03_Socket, J10 Conn_01x04_Pin, J2 Conn_01x03_Socket, J3 Motor1, J4 Motor2, J5 Motor3, J6 Motor4, J7 Conn_01x04_Pin, J8 Conn_01x04_Pin, J9 Conn_01x04_Pin, U3 ROB-14450, U4 ESP32-DevKitC, U5 ROB-14450

Commit message: майже готова PCB
Parts:
- U1: footprint BMS ROS2 project:Untitled -> BMS ROS2 project:BMS ROS2 project
- U2: footprint BMS ROS2 project:Untitled -> BMS ROS2 project:Buck convertor
Changed lines of the file:
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@@
 		)
 	)
-	(footprint "BMS ROS2 project:Untitled"
+	(footprint "BMS ROS2 project:BMS ROS2 project"
 		(layer "F.Cu")
 		(at 150.82 50.89 180)
@@
 		)
 	)
-	(footprint "BMS ROS2 project:Untitled"
+	(footprint "BMS ROS2 project:Buck convertor"
 		(layer "F.Cu")
 		(at 205.82 75.62 -90)

Commit message: Add files via upload
Parts:
- removed U5: ROB-14450, ROB-14450:MODULE_ROB-14450
- added C10: 20u, Capacitor_THT:C_Disc_D4.3mm_W1.9mm_P5.00mm, F.Cu at (168.8, 73.8)
- added C11: 20u, Capacitor_THT:C_Disc_D4.3mm_W1.9mm_P5.00mm, F.Cu at (144.8, 73.4)
- added C4: 220uF, Capacitor_THT:CP_Radial_D13.0mm_P5.00mm, F.Cu at (168.8, 76.5)
- added C5: 220uF, Capacitor_THT:CP_Radial_D13.0mm_P5.00mm, F.Cu at (168.8, 104.3)
- added C6: 20u, Capacitor_THT:C_Disc_D4.3mm_W1.9mm_P5.00mm, F.Cu at (168.8, 101.7)
- added C7: 20u, Capacitor_THT:C_Disc_D4.3mm_W1.9mm_P5.00mm, F.Cu at (144.7, 101.7)
- added C8: 220uF, Capacitor_THT:CP_Radial_D13.0mm_P5.00mm, F.Cu at (144.9, 104.4)
- added C9: 220uF, Capacitor_THT:CP_Radial_D13.0mm_P5.00mm, F.Cu at (144.7, 76.5)
- added D1: LED, LED_THT:LED_D3.0mm, F.Cu at (77.0, 79.1)
- added J11: switch, Connector_Molex:Molex_KK-254_AE-6410-02A_1x02_P2.54mm_Vertical, F.Cu at (134.2, 51.8)
- added R1: 560R, Resistor_THT:R_Axial_DIN0204_L3.6mm_D1.6mm_P7.62mm_Horizontal, F.Cu at (77.1, 68.1)
- added U6: ROB-14450, ROB-14450:MODULE_ROB-14450, F.Cu at (166.2, 113.4)
- added U7: ROB-14450, ROB-14450:MODULE_ROB-14450, F.Cu at (166.3, 85.6)
- added U8: ROB-14450, ROB-14450:MODULE_ROB-14450, F.Cu at (142.3, 113.3)
- added U9: ROB-14450, ROB-14450:MODULE_ROB-14450, F.Cu at (142.1, 85.5)
- C1: value 2200nF -> 10uF; footprint Capacitor_THT:C_Radial_D12.5mm_H20.0mm_P5.00mm -> Capacitor_THT:C_Disc_D3.0mm_W1.6mm_P2.50mm
- C2: footprint Capacitor_THT:C_Disc_D8.0mm_W5.0mm_P7.50mm -> Capacitor_THT:C_Disc_D3.0mm_W1.6mm_P2.50mm
- C3: value 10uF -> 2200nF; footprint Capacitor_THT:C_Disc_D8.0mm_W5.0mm_P7.50mm -> Capacitor_THT:C_Radial_D12.5mm_H20.0mm_P5.00mm
- J1: value Conn_01x03_Socket -> Conn_01x04_Pin; footprint Connector_PinSocket_2.00mm:PinSocket_1x03_P2.00mm_Vertical -> Connector_JST:JST_PH_B4B-PH-K_1x04_P2.00mm_Vertical
- J10: value Conn_01x04_Pin -> Motor3; footprint Connector_JST:JST_PH_B4B-PH-K_1x04_P2.00mm_Vertical -> Connector_Molex:Molex_KK-254_AE-6410-02A_1x02_P2.54mm_Vertical
- J2: value Conn_01x03_Socket -> Conn_01x04_Pin; footprint Connector:FanPinHeader_1x03_P2.54mm_Vertical -> Connector_JST:JST_PH_B4B-PH-K_1x04_P2.00mm_Vertical
- J3: value Motor1 -> Conn_01x03_Socket; footprint Connector_Molex:Molex_KK-254_AE-6410-02A_1x02_P2.54mm_Vertical -> Connector:FanPinHeader_1x03_P2.54mm_Vertical
- J4: value Motor2 -> Conn_01x04_Pin; footprint Connector_Molex:Molex_KK-254_AE-6410-02A_1x02_P2.54mm_Vertical -> Connector_JST:JST_PH_B4B-PH-K_1x04_P2.00mm_Vertical
- J5: value Motor3 -> Conn_01x04_Pin; footprint Connector_Molex:Molex_KK-254_AE-6410-02A_1x02_P2.54mm_Vertical -> Connector_JST:JST_PH_B4B-PH-K_1x04_P2.00mm_Vertical
- J6: value Motor4 -> Conn_01x03_Socket; footprint Connector_Molex:Molex_KK-254_AE-6410-02A_1x02_P2.54mm_Vertical -> Connector_PinSocket_2.00mm:PinSocket_1x03_P2.00mm_Vertical
- J7: value Conn_01x04_Pin -> Motor1; footprint Connector_JST:JST_PH_B4B-PH-K_1x04_P2.00mm_Vertical -> Connector_Molex:Molex_KK-254_AE-6410-02A_1x02_P2.54mm_Vertical
- J8: value Conn_01x04_Pin -> Motor4; footprint Connector_JST:JST_PH_B4B-PH-K_1x04_P2.00mm_Vertical -> Connector_Molex:Molex_KK-254_AE-6410-02A_1x02_P2.54mm_Vertical
- J9: value Conn_01x04_Pin -> Motor2; footprint Connector_JST:JST_PH_B4B-PH-K_1x04_P2.00mm_Vertical -> Connector_Molex:Molex_KK-254_AE-6410-02A_1x02_P2.54mm_Vertical
- U3: value ROB-14450 -> ESP32-DevKitC; footprint ROB-14450:MODULE_ROB-14450 -> PCM_Espressif:ESP32-DevKitC
- U4: value ESP32-DevKitC -> ZC323900; footprint PCM_Espressif:ESP32-DevKitC -> ZC323900:MODULE_ZC323900
- moved J4 135.9 mm to (75.5, 100.9)
- moved J1 120.1 mm to (75.5, 111.9), turned to 90 degrees
- moved U2 116.2 mm to (90.9, 58.4), turned to 180 degrees
- moved U3 115.5 mm to (82.8, 78.3), turned to 0 degrees
- moved C2 100.7 mm to (111.2, 62.4), turned to 180 degrees
- moved C1 93.3 mm to (111.3, 52.9)
- moved C3 91.0 mm to (119.9, 52.1), turned to -90 degrees
- moved J2 58.8 mm to (75.5, 89.9)
- moved J5 57.3 mm to (75.5, 122.9)
- moved U4 52.7 mm to (120.4, 112.0)
- moved J3 48.0 mm to (192.1, 57.1)
- moved J6 34.4 mm to (113.8, 66.4), turned to 0 degrees
- moved J10 34.1 mm to (181.5, 107.3)
- moved J9 33.5 mm to (181.6, 84.3), turned to -90 degrees
- moved U1 15.6 mm to (163.6, 59.8), turned to 0 degrees
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Connections:
- C1 pad 1: VCC -> GNDD
- C1 pad 2: GNDD -> VCC
- C3 pad 1: GNDD -> VCC
- C3 pad 2: VCC -> GNDD
- J1 pad 2: /BAT_LVL_OUT -> GNDD
- J1 pad 3: GNDD -> Net-(J1-Pin_3)
- J10 pad 1: +5V -> Net-(J10-Pin_1)
- J10 pad 2: GNDD -> Net-(J10-Pin_2)
- J2 pad 1: Net-(J2-Pin_1) -> +5V
- J2 pad 2: Net-(J2-Pin_2) -> GNDD
- J4 pad 1: Net-(J4-Pin_1) -> +5V
- J4 pad 2: Net-(J4-Pin_2) -> GNDD
- J5 pad 1: Net-(J5-Pin_1) -> +5V
- J5 pad 2: Net-(J5-Pin_2) -> GNDD
- J6 pad 1: Net-(J6-Pin_1) -> +5V
- J6 pad 2: Net-(J6-Pin_2) -> /BAT_LVL_OUT
- J7 pad 1: +5V -> Net-(J7-Pin_1)
- J7 pad 2: GNDD -> Net-(J7-Pin_2)
- J8 pad 1: +5V -> Net-(J8-Pin_1)
- J8 pad 2: GNDD -> Net-(J8-Pin_2)
- J9 pad 1: +5V -> Net-(J9-Pin_1)
- J9 pad 2: GNDD -> Net-(J9-Pin_2)
- U1 pad 2: VCC -> Net-(J11-Pin_1)
- U1 pad 3: Net-(J2-Pin_1) -> Net-(J3-Pin_1)
- U1 pad 4: Net-(J2-Pin_2) -> Net-(J3-Pin_2)
- U1 pad 5: Net-(J2-Pin_3) -> Net-(J3-Pin_3)
- U3 pad 1: VCC -> +3.3V
- U3 pad 10: /PWM_M2 -> unconnected-(U3-DAC_2/ADC2_CH9/GPIO26-Pad10)
- U3 pad 11: /M2_AI2 -> unconnected-(U3-ADC2_CH7/GPIO27-Pad11)
- U3 pad 12: /M2_AI1 -> unconnected-(U3-MTMS/GPIO14/ADC2_CH6-Pad12)
- U3 pad 13: +5V -> Net-(J1-Pin_4)
- U3 pad 14: /M1_AI1 -> GNDD
- U3 pad 15: /M1_AI2 -> Net-(J1-Pin_3)
- U3 pad 16: /PWM_M1 -> Net-(J5-Pin_4)
- U3 pad 2: +5V -> unconnected-(U3-CHIP_PU-Pad2)
- U3 pad 3: GNDD -> Net-(J2-Pin_4)
- U3 pad 4: Net-(J3-Pin_2) -> Net-(J2-Pin_3)
- U3 pad 5: Net-(J3-Pin_1) -> unconnected-(U3-VDET_1/GPIO34/ADC1_CH6-Pad5)
- U3 pad 6: Net-(J4-Pin_1) -> unconnected-(U3-VDET_2/GPIO35/ADC1_CH7-Pad6)
- U3 pad 7: Net-(J4-Pin_2) -> Net-(J4-Pin_3)
- U3 pad 8: GNDD -> Net-(J4-Pin_4)
- U3 pad 9: GNDD -> unconnected-(U3-DAC_1/ADC2_CH8/GPIO25-Pad9)
- U4 pad 1: unconnected-(U4-3V3-Pad1) -> +3.3V
- U4 pad 10: /M4_AI1 -> +3.3V
- U4 pad 11: /M4_AI2 -> GNDD
- U4 pad 12: /PWM_M4 -> /M4_AI2
- U4 pad 13: Net-(J8-Pin_4) -> /M4_AI1
- U4 pad 14: GNDD -> /M3_AI2
- U4 pad 15: Net-(J8-Pin_3) -> /M3_AI1
- U4 pad 16: Net-(J10-Pin_4) -> /M2_AI2
- U4 pad 17: Net-(J10-Pin_3) -> /M2_AI1
- U4 pad 18: unconnected-(U4-CMD-Pad18) -> /M1_AI2
- U4 pad 19: +5V -> /M1_AI1
- U4 pad 2: unconnected-(U4-CHIP_PU-Pad2) -> /M1_AI1_3.3
- U4 pad 20: unconnected-(U4-SD_CLK/GPIO6-Pad20) -> +5V
- U4 pad 3: Net-(J9-Pin_4) -> /M1_AI2_3.3
- U4 pad 4: Net-(J9-Pin_3) -> /M2_AI1_3.3
- U4 pad 5: unconnected-(U4-VDET_1/GPIO34/ADC1_CH6-Pad5) -> /M2_AI2_3.3
- U4 pad 6: /PWM_M3 -> /M3_AI1_3.3
- U4 pad 7: /M3_AI2 -> /M3_AI2_3.3
- U4 pad 8: /M3_AI1 -> /M4_AI1_3.3
- U4 pad 9: /BAT_LVL_OUT -> /M4_AI2_3.3
Routing:
- net +5V: track 229.8 -> 45.0 mm
- net VCC: track 149.3 -> 250.8 mm
- net +3.3V: track 0.00 -> 92.6 mm
- net Net-(J10-Pin_2): track 0.00 -> 51.5 mm
- net /M2_AI2: track 7.42 -> 58.7 mm
- net Net-(J7-Pin_2): track 0.00 -> 51.3 mm
- net /M2_AI1: track 7.42 -> 52.9 mm
- net Net-(J10-Pin_1): track 0.00 -> 44.5 mm
- net /M4_AI2: track 6.71 -> 50.5 mm
- net Net-(J7-Pin_1): track 0.00 -> 43.0 mm
- net Net-(J8-Pin_3): track 42.3 -> 0.00 mm
- net Net-(J8-Pin_4): track 40.7 -> 0.00 mm
- net /M4_AI1: track 6.71 -> 45.1 mm
- net /M1_AI2: track 7.42 -> 45.7 mm
- net /BAT_LVL_OUT: track 43.2 -> 15.6 mm
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
Commit message: Add files via upload
Parts:
- moved D1 0.84 mm to (77.8, 79.1)
- moved J1 0.78 mm to (76.3, 111.9)
- moved J2 0.78 mm to (76.3, 89.9)
- moved J4 0.78 mm to (76.3, 100.9)
- moved J5 0.78 mm to (76.3, 122.9)
Connections:
- U3 pad 12: unconnected-(U3-MTMS/GPIO14/ADC2_CH6-Pad12) -> Net-(J1-Pin_4)
- U3 pad 13: Net-(J1-Pin_4) -> Net-(J1-Pin_3)
- U3 pad 15: Net-(J1-Pin_3) -> /GPIO13
- U3 pad 30: /PWM_M1 -> /PWM_M4
- U3 pad 31: /PWM_M2 -> /PWM_M3
- U3 pad 33: /PWM_M3 -> /PWM_M2
- U3 pad 36: /PWM_M4 -> /PWM_M1
- U3 pad 7: Net-(J4-Pin_3) -> Net-(J4-Pin_4)
- U3 pad 8: Net-(J4-Pin_4) -> Net-(J4-Pin_3)
Routing:
- net GNDD: track 37.6 -> 515.2 mm, vias 0 -> 1
- net +5V: track 45.0 -> 378.5 mm
- net /PWM_M4: track 20.3 -> 99.5 mm
- net /PWM_M2: track 21.5 -> 75.2 mm
- net /PWM_M3: track 20.4 -> 56.5 mm
- net /PWM_M1: track 26.8 -> 49.0 mm
- net VCC: track 250.8 -> 234.5 mm
- net Net-(J4-Pin_4): track 0.00 -> 7.08 mm
- net Net-(J4-Pin_3): track 0.00 -> 6.85 mm
- net Net-(J1-Pin_4): track 0.48 -> 6.65 mm
- net Net-(J1-Pin_3): track 0.70 -> 6.87 mm
- net +3.3V: track 92.6 -> 97.8 mm
- net Net-(D1-A): track 0.01 -> 4.17 mm
- net Net-(J5-Pin_4): track 7.49 -> 6.71 mm
- net Net-(J2-Pin_4): track 7.51 -> 6.73 mm
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
Commit message: Покращення
Parts:
- added J12: Conn_01x04_Pin, Connector_PinHeader_2.54mm:PinHeader_1x04_P2.54mm_Vertical, F.Cu at (114.2, 80.0)
- added J13: Conn_01x04_Pin, Connector_PinHeader_2.54mm:PinHeader_1x04_P2.54mm_Vertical, F.Cu at (85.2, 131.0)
- added J14: Conn_01x04_Pin, Connector_PinHeader_2.54mm:PinHeader_1x04_P2.54mm_Vertical, F.Cu at (97.5, 131.0)
- added R2: 10К, Resistor_THT:R_Axial_DIN0204_L3.6mm_D1.6mm_P5.08mm_Horizontal, F.Cu at (91.5, 74.0)
- moved R1 7.54 mm to (82.8, 73.0), turned to 180 degrees
Connections:
- U3 pad 10: unconnected-(U3-DAC_2/ADC2_CH9/GPIO26-Pad10) -> Net-(J13-Pin_3)
- U3 pad 11: unconnected-(U3-ADC2_CH7/GPIO27-Pad11) -> Net-(J13-Pin_2)
- U3 pad 15: /GPIO13 -> Net-(J13-Pin_1)
- U3 pad 2: unconnected-(U3-CHIP_PU-Pad2) -> Net-(U3-CHIP_PU)
- U3 pad 28: unconnected-(U3-GPIO17-Pad28) -> Net-(J14-Pin_4)
- U3 pad 29: unconnected-(U3-GPIO5-Pad29) -> Net-(J12-Pin_4)
- U3 pad 34: unconnected-(U3-U0RXD/GPIO3-Pad34) -> Net-(J12-Pin_3)
- U3 pad 35: unconnected-(U3-U0TXD/GPIO1-Pad35) -> Net-(J12-Pin_2)
- U3 pad 5: unconnected-(U3-VDET_1/GPIO34/ADC1_CH6-Pad5) -> Net-(J14-Pin_2)
- U3 pad 6: unconnected-(U3-VDET_2/GPIO35/ADC1_CH7-Pad6) -> Net-(J14-Pin_1)
- U3 pad 9: unconnected-(U3-DAC_1/ADC2_CH8/GPIO25-Pad9) -> Net-(J13-Pin_4)
Routing:
- net Net-(J14-Pin_2): track 0.00 -> 50.2 mm
- net Net-(J14-Pin_1): track 0.00 -> 46.8 mm
- net Net-(J13-Pin_4): track 0.00 -> 37.2 mm
- net Net-(J13-Pin_3): track 0.00 -> 34.6 mm
- net Net-(J13-Pin_2): track 0.00 -> 32.6 mm
- net Net-(J14-Pin_4): track 0.00 -> 29.0 mm
- net Net-(J12-Pin_4): track 0.00 -> 27.2 mm
- net Net-(J13-Pin_1): track 0.00 -> 19.3 mm
- net Net-(J12-Pin_3): track 0.00 -> 15.6 mm
- net Net-(J12-Pin_2): track 0.00 -> 13.3 mm
- net Net-(U3-CHIP_PU): track 0.00 -> 11.6 mm
- net Net-(D1-A): track 4.17 -> 10.3 mm
- net +3.3V: track 97.8 -> 103.6 mm
- net +5V: track 378.5 -> 382.5 mm
- net unconnected-(U3-CMD-Pad18): track 0.00 -> 1.18 mm
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Other:
- board text added: "1"
- board text added: "13"
- board text added: "17"
- board text added: "25"
- board text added: "26"
- board text added: "27"
- board text added: "3"
- board text added: "34"
- board text added: "35"
- board text added: "5"
